File: minimal_adp1074/minimal_adp1074.kicad_pcb (KiCad board)
At the start: 4 copper layers, 25.4 x 25.4 mm, 0 parts

Commit message: backup
Parts:
- added T1: PL160X9-102L-BLD, transformer_footprints:PL160X9-102L, F.Cu at (152.4, 88.9)
- added U1: ADP1074ACCZ-R7, analog_devices_footprints:CC-24-6_ADI, F.Cu at (152.4, 103.5)
Routing:
- added copper zone on B.Cu, net GND
- added copper zone on F.Cu, net GND
- added copper zone on In1.Cu, net GND
- added copper zone on In2.Cu, net GND
- added copper zone on B.Cu, net GNDA
- added copper zone on F.Cu, net GNDA
- added copper zone on In1.Cu, net GNDA
- added copper zone on In2.Cu, net GNDA
Other:
- board size 25.4 x 25.4 mm -> 38.1 x 30.5 mm

Commit message: backup
Parts:
- added D1: 100 V, diode_footprints:SOD323, F.Cu at (137.9, 81.0)
- added D2: 100 V, diode_footprints:SOD323, F.Cu at (137.9, 79.3)
- added L1: 1000.0 µH, inductor_footprints:CB2518T, F.Cu at (134.5, 80.1)
Connections:
- T1 pad 1: unconnected-(T1-Pad1) -> Net-(D1-Pad2)
- T1 pad 6: unconnected-(T1-Pad6) -> Net-(D2-Pad2)
Routing:
- net Net-(D2-Pad2): track 0.00 -> 22.6 mm
- net Net-(D1-Pad2): track 0.00 -> 2.97 mm
- added copper zone on F.Cu, net Net-(D1-Pad1)
Other:
- board size 38.1 x 30.5 mm -> 43.2 x 30.5 mm

Commit message: backup
Parts:
- added C1: 2.2 µF, capacitor_footprints:C_0805_2012Metric, F.Cu at (131.7, 81.3)
- added C2: 2.2 µF, capacitor_footprints:C_1206_3216Metric, F.Cu at (133.1, 86.1)
- added C3: 2.2 µF, capacitor_footprints:C_1206_3216Metric, F.Cu at (135.8, 86.1)
- added C4: 2.2 µF, capacitor_footprints:C_1206_3216Metric, F.Cu at (138.5, 86.1)
- added D3: 11.0 V, diode_footprints:SOD_123, F.Cu at (129.3, 80.6)
- added Q1: 80 V, transistor_footprints:PowerPAK SO-8 Single, F.Cu at (137.1, 93.8)
- added R1: 100 Ω, resistor_footprints:R_0402_1005Metric, F.Cu at (131.7, 78.9)
Connections:
- D2 pad 2: Net-(D2-Pad2) -> GND
- L1 pad 2: unconnected-(L1-Pad2) -> /V_AUX
- T1 pad 6: Net-(D2-Pad2) -> GND
- U1 pad 1: unconnected-(U1-NGATE-Pad1) -> /N_GATE
Routing:
- net Net-(D2-Pad2): track 22.6 -> 0.00 mm
- net Net-(D3-Pad1): track 0.00 -> 1.85 mm
- added copper zone on F.Cu, net /VIN
- added copper zone on F.Cu, net /V_AUX
Other:
- board size 43.2 x 30.5 mm -> 50.8 x 30.5 mm

Commit message: backup
Parts:
- added C5: 100 nF, capacitor_footprints:C_0402_1005Metric, F.Cu at (147.1, 102.2)
- added C6: 2.2 µF, capacitor_footprints:C_0603_1608Metric, F.Cu at (158.0, 102.0)
- added C7: 220 nF, capacitor_footprints:C_0603_1608Metric, F.Cu at (137.1, 95.5)
- added C8: 100 nF, capacitor_footprints:C_0402_1005Metric, F.Cu at (139.0, 96.3)
- added C9: 100 nF, capacitor_footprints:C_0402_1005Metric, F.Cu at (136.5, 101.2)
- added D4: 100 V, diode_footprints:SOD323, F.Cu at (138.1, 102.7)
- added D5: 11.0 V, diode_footprints:SOD_123, F.Cu at (142.6, 102.3)
- added L2: 2.0 µH, inductor_footprints:IHLP4040DZE_V2, F.Cu at (170.9, 88.9)
- added Q2: -60 V, transistor_footprints:SOT-26, F.Cu at (138.2, 98.9)
- added R2: 0.008 Ω, resistor_footprints:R_1206_3216Metric, F.Cu at (130.6, 99.8)
- added R3: 10 kΩ, resistor_footprints:R_0402_1005Metric, F.Cu at (134.4, 98.0)
- added R4: 0 Ω, resistor_footprints:R_0402_1005Metric, F.Cu at (134.4, 99.3)
- added R5: 1.5 kΩ, resistor_footprints:R_0402_1005Metric, F.Cu at (132.5, 98.6)
- added R6: 10 kΩ, resistor_footprints:R_0402_1005Metric, F.Cu at (138.6, 101.2)
- added R7: 1 kΩ, resistor_footprints:R_0402_1005Metric, F.Cu at (139.0, 95.1)
- added R8: 10 kΩ, resistor_footprints:R_0402_1005Metric, F.Cu at (140.9, 103.4)
- C1: footprint capacitor_footprints:C_0805_2012Metric -> capacitor_footprints:C_0603_1608Metric
- moved Q1 5.13 mm to (132.0, 93.8)
- moved R1 1.43 mm to (132.9, 78.2)
- moved D3 0.98 mm to (129.9, 79.8)
- moved C2 0.25 mm to (132.9, 86.1)
- moved C1 0.25 mm to (131.9, 81.3)
- moved C3 0.13 mm to (135.7, 86.1)
Connections:
- C1 pad 2: /V_AUX -> /VREG1
- L1 pad 2: /V_AUX -> /VREG1
- Q1 pad 1: unconnected-(Q1-S-Pad1) -> Net-(Q1-S-Pad1)
- Q1 pad 2: unconnected-(Q1-S-Pad2) -> Net-(Q1-S-Pad1)
- Q1 pad 3: unconnected-(Q1-S-Pad3) -> Net-(Q1-S-Pad1)
- Q1 pad 4: /N_GATE -> Net-(Q1-G)
- R1 pad 1: /V_AUX -> /VREG1
- T1 pad 7: unconnected-(T1-Pad7) -> Net-(L2-Pad1)
- U1 pad 2: unconnected-(U1-PGATE-Pad2) -> /P_GATE
- U1 pad 20: unconnected-(U1-VREG2-Pad20) -> /VERG2
- U1 pad 5: unconnected-(U1-VREG1-Pad5) -> /VREG1
- U1 pad 8: unconnected-(U1-CS-Pad8) -> /CS
Routing:
- net /VREG1: track 0.00 -> 36.8 mm, vias 0 -> 2
- net /CS: track 0.00 -> 18.6 mm, vias 0 -> 2
- net /N_GATE: track 0.00 -> 17.9 mm, vias 0 -> 2
- net /P_GATE: track 0.00 -> 15.5 mm, vias 0 -> 2
- net Net-(Q2-G): track 0.00 -> 3.95 mm
- net Net-(Q1-G): track 0.00 -> 2.87 mm
- net Net-(D5-Pad1): track 0.00 -> 1.72 mm
- net /VERG2: track 0.00 -> 1.58 mm
- net Net-(C8-Pad1): track 0.00 -> 1.18 mm
- net /VIN: track 0.00 -> 0.76 mm, vias 0 -> 16
- net Net-(D3-Pad1): track 1.85 -> 2.45 mm
- net GND: vias 0 -> 18
- added copper zone on In1.Cu, net /VIN
- added copper zone on F.Cu, net /VREG1
- added copper zone on F.Cu, net Net-(C7-Pad2)
- added copper zone on F.Cu, net Net-(Q1-D)
- added copper zone on F.Cu, net Net-(Q1-S-Pad1)
- removed copper zone on F.Cu, net /V_AUX
- removed copper zone on In1.Cu, net GND

Commit message: backup
Parts:
- added C10: 10 nF, capacitor_footprints:C_0402_1005Metric, F.Cu at (170.7, 80.9)
- added C11: 10 nF, capacitor_footprints:C_0402_1005Metric, F.Cu at (170.7, 101.4)
- added D6: 100 V, diode_footprints:SOD323, F.Cu at (168.0, 80.9)
- added D7: 100 V, diode_footprints:SOD323, F.Cu at (168.0, 101.4)
- added Q3: 40 V, transistor_footprints:TDSON-8 FL, F.Cu at (168.4, 77.4)
- added Q4: 40 V, transistor_footprints:TDSON-8 FL, F.Cu at (168.4, 97.9)
- added R10: 10 kΩ, resistor_footprints:R_0402_1005Metric, F.Cu at (173.2, 75.5)
- added R11: 10 kΩ, resistor_footprints:R_0402_1005Metric, F.Cu at (173.2, 96.0)
- added R12: 0 Ω, resistor_footprints:R_0402_1005Metric, F.Cu at (173.2, 97.3)
- added R13: 10 kΩ, resistor_footprints:R_0402_1005Metric, F.Cu at (170.7, 82.2)
- added R14: 10 kΩ, resistor_footprints:R_0402_1005Metric, F.Cu at (170.7, 102.7)
- added R9: 0 Ω, resistor_footprints:R_0402_1005Metric, F.Cu at (173.2, 76.8)
- L2: value 2.0 µH -> 2.2 µH; footprint inductor_footprints:IHLP4040DZE_V2 -> inductor_footprints:74439369
Connections:
- net Net-(Q1-G) renamed /N_GATE_G
- net Net-(Q2-G) renamed /P_GATE_G
- T1 pad 11: unconnected-(T1-Pad11) -> Net-(Q3-D)
- U1 pad 23: unconnected-(U1-SR2-Pad23) -> /SR2
- U1 pad 24: unconnected-(U1-SR1-Pad24) -> /SR1
Routing:
- net /SR1: track 0.00 -> 35.8 mm, vias 0 -> 2
- net /SR2: track 0.00 -> 22.4 mm, vias 0 -> 2
- net /SR1_G: track 0.00 -> 2.85 mm
- net /SR2_G: track 0.00 -> 2.84 mm
- net Net-(C10-Pad1): track 0.00 -> 2.35 mm
- net Net-(C11-Pad1): track 0.00 -> 2.35 mm
- net /VOUT: track 0.00 -> 1.52 mm, vias 0 -> 22
- net /P_GATE: track 15.5 -> 16.5 mm
- net /N_GATE: track 17.9 -> 18.5 mm
- net GNDA: vias 0 -> 4
- added copper zone on F.Cu, net /VOUT
- added copper zone on In1.Cu, net /VOUT
- added copper zone on F.Cu, net Net-(Q3-D)
- added copper zone on F.Cu, net Net-(Q4-D)
- removed copper zone on In1.Cu, net GNDA
Other:
- board size 50.8 x 30.5 mm -> 50.8 x 35.6 mm

Commit message: backup
Parts:
- added C12: 220 µF, capacitor_footprints:C_1206_3216Metric, F.Cu at (178.6, 86.3)
- added C13: 220 µF, capacitor_footprints:C_1206_3216Metric, F.Cu at (178.6, 91.4)
- added C14: 220 µF, capacitor_footprints:C_1206_3216Metric, F.Cu at (181.4, 86.3)
- added C15: 220 µF, capacitor_footprints:C_1206_3216Metric, F.Cu at (184.2, 86.3)
- added C16: 220 µF, capacitor_footprints:C_1206_3216Metric, F.Cu at (181.4, 91.4)
- added C17: 220 µF, capacitor_footprints:C_1206_3216Metric, F.Cu at (184.2, 91.4)
- added C18: 1.5 µF, capacitor_footprints:C_0603_1608Metric, F.Cu at (147.8, 108.8)
- added C19: 100 nF, capacitor_footprints:C_0402_1005Metric, F.Cu at (156.3, 107.8)
- added C20: 100 pF, capacitor_footprints:C_0402_1005Metric, F.Cu at (158.3, 108.8)
- added C21: 4.7 nF, capacitor_footprints:C_0402_1005Metric, F.Cu at (158.3, 107.5)
- added R15: 28 kΩ, resistor_footprints:R_0402_1005Metric, F.Cu at (146.7, 105.6)
- added R16: 49.9 kΩ, resistor_footprints:R_0402_1005Metric, F.Cu at (150.0, 108.1)
- added R17: 0 Ω, resistor_footprints:R_0402_1005Metric, F.Cu at (147.5, 107.3)
- added R18: 10 kΩ, resistor_footprints:R_0402_1005Metric, F.Cu at (155.6, 109.8)
- added R19: 0 Ω, resistor_footprints:R_0402_1005Metric, F.Cu at (154.8, 107.8)
- added R20: 24.9 kΩ, resistor_footprints:R_0402_1005Metric, F.Cu at (160.1, 108.0)
- added R21: 3.16 kΩ, resistor_footprints:R_0402_1005Metric, F.Cu at (158.5, 105.9)
- added R22: 976 Ω, resistor_footprints:R_0402_1005Metric, F.Cu at (160.2, 105.4)
- added R23: 3.09 kΩ, resistor_footprints:R_0402_1005Metric, F.Cu at (158.5, 103.5)
- added R24: 887 Ω, resistor_footprints:R_0402_1005Metric, F.Cu at (160.2, 104.0)
- moved R14 5.36 mm to (167.8, 107.2)
- moved C11 5.36 mm to (167.8, 105.9)
- moved Q4 5.36 mm to (165.5, 102.4)
- moved R11 5.36 mm to (170.3, 100.5)
- moved D7 5.36 mm to (165.1, 105.9)
- moved R12 5.36 mm to (170.3, 101.8)
- moved R9 3.29 mm to (173.2, 80.1)
- moved C10 3.29 mm to (170.7, 84.2)
- moved D6 3.29 mm to (168.0, 84.2)
- moved Q3 3.29 mm to (168.4, 80.7)
- moved R10 3.29 mm to (173.2, 78.7)
- moved R13 3.29 mm to (170.7, 85.5)
- moved L2 3.15 mm to (170.9, 92.0)
- moved C6 1.51 mm to (158.6, 100.6), turned to 0 degrees
Connections:
- net /VERG2 renamed /VREG2
- U1 pad 10: unconnected-(U1-SYNC-Pad10) -> /SYNC
- U1 pad 11: unconnected-(U1-SS1-Pad11) -> /SS1
- U1 pad 12: unconnected-(U1-DMAX-Pad12) -> /DMAX
- U1 pad 13: unconnected-(U1-MODE-Pad13) -> /MODE
- U1 pad 14: unconnected-(U1-~{PGOOD}-Pad14) -> /~{PGOOD}
- U1 pad 15: unconnected-(U1-SS2-Pad15) -> /SS2
- U1 pad 16: unconnected-(U1-COMP-Pad16) -> /COMP
- U1 pad 17: unconnected-(U1-FB-Pad17) -> /FB
- U1 pad 18: unconnected-(U1-OVP-Pad18) -> /OVP
- U1 pad 9: unconnected-(U1-RT-Pad9) -> /RT
Routing:
- net /VREG2: track 1.58 -> 17.9 mm, vias 0 -> 2
- net /DMAX: track 0.00 -> 5.68 mm, vias 0 -> 2
- net /COMP: track 0.00 -> 5.00 mm
- net /SR2: track 22.4 -> 17.6 mm
- net /~{PGOOD}: track 0.00 -> 4.68 mm
- net /SS1: track 0.00 -> 3.73 mm
- net /FB: track 0.00 -> 3.67 mm
- net /OVP: track 0.00 -> 3.33 mm
- net /VREG1: track 36.8 -> 34.1 mm
- net /SYNC: track 0.00 -> 2.19 mm
- net /SS2: track 0.00 -> 2.09 mm
- net /MODE: track 0.00 -> 1.84 mm
- net /RT: track 0.00 -> 1.76 mm, vias 0 -> 1
- net /VOUT: track 1.52 -> 3.05 mm, vias 22 -> 36
- net /SR1: track 35.8 -> 34.4 mm
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Other:
- board size 50.8 x 35.6 mm -> 59.7 x 35.6 mm

Commit message: backup
Parts:
- added C22: 1.5 µF, capacitor_footprints:C_0603_1608Metric, F.Cu at (159.8, 102.1)
- added C23: 1.5 µF, capacitor_footprints:C_0603_1608Metric, F.Cu at (161.6, 102.1)
- added D8: 100 V, diode_footprints:SOD323, F.Cu at (163.3, 102.1)
- moved C11 3.22 mm to (170.7, 104.6)
- moved R14 3.22 mm to (170.7, 105.9)
- moved Q4 3.22 mm to (168.4, 101.1)
- moved D7 3.22 mm to (168.0, 104.6)
- moved R11 3.22 mm to (173.2, 99.2)
- moved R12 3.22 mm to (173.2, 100.5)
- moved R22 2.34 mm to (161.8, 107.0), turned to -90 degrees
- moved R23 2.13 mm to (160.2, 104.8), turned to 90 degrees
- moved R21 2.07 mm to (160.2, 107.0)
- moved C20 1.87 mm to (157.7, 107.0), turned to -90 degrees
- moved R24 1.80 mm to (161.8, 104.8), turned to -90 degrees
- moved C6 1.63 mm to (158.0, 102.1), turned to 90 degrees
- moved R20 1.52 mm to (159.0, 109.1)
- moved C19 1.40 mm to (156.9, 109.1)
- moved R18 1.40 mm to (156.1, 111.1), turned to 0 degrees
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Connections:
- net Net-(Q4-D) renamed /SW
- U1 pad 19: unconnected-(U1-VDD2-Pad19) -> /VDD2
Routing:
- net /VDD2: track 0.00 -> 7.35 mm
- net /SR2: track 17.6 -> 21.5 mm
- net /COMP: track 5.00 -> 2.91 mm
- net /FB: track 3.67 -> 5.68 mm
- net /OVP: track 3.33 -> 5.24 mm
- net /VREG2: track 17.9 -> 16.3 mm
- net /SR1: track 34.4 -> 33.6 mm
- net /N_GATE: track 18.5 -> 17.8 mm
- net GNDA: vias 32 -> 41
Other:
- board size 59.7 x 35.6 mm -> 59.7 x 36.8 mm

Commit message: backup
Parts:
- added D10: 40 V, diode_footprints:SMA, F.Cu at (168.4, 110.3)
- added D9: 40 V, diode_footprints:SMA, F.Cu at (169.9, 87.0)
- moved C11 3.09 mm to (170.7, 107.6), turned to 90 degrees
- moved D7 3.09 mm to (168.0, 107.6)
- moved C12 2.88 mm to (178.6, 89.2)
- moved C13 2.88 mm to (178.6, 94.3)
- moved C14 2.88 mm to (181.4, 89.2)
- moved C15 2.88 mm to (184.2, 89.2)
- moved C16 2.88 mm to (181.4, 94.3)
- moved C17 2.88 mm to (184.2, 94.3)
- moved L2 2.88 mm to (170.9, 94.9)
- moved Q4 2.88 mm to (168.4, 103.9)
- moved R12 2.88 mm to (173.2, 103.3)
- moved R11 2.88 mm to (173.2, 102.0)
- moved R14 2.40 mm to (172.4, 107.6), turned to -90 degrees
- moved R13 2.00 mm to (172.4, 84.3), turned to -90 degrees
- moved D6 0.27 mm to (168.2, 84.4)
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Routing:
- net Net-(C11-Pad1): track 2.35 -> 3.32 mm
- net Net-(C10-Pad1): track 2.35 -> 3.14 mm
- net GNDA: vias 41 -> 47
