File: minimal_adp1074/minimal_adp1074.kicad_pcb (KiCad board)
At the start: 4 copper layers, 59.7 x 36.8 mm, 65 parts, among them Q1 80 V, Q2 -60 V, Q3 40 V, Q4 40 V, T1 PL160X9-102L-BLD, U1 ADP1074ACCZ-R7

Commit message: backup
Parts:
- added C24: 2.2 µF, capacitor_footprints:C_0603_1608Metric, F.Cu at (144.6, 103.5)
- added C25: 2.2 µF, capacitor_footprints:C_0603_1608Metric, F.Cu at (142.9, 103.5)
- added Q5: 150 V, transistor_footprints:SOT23-3, F.Cu at (141.9, 106.8)
- added R25: 24.3 kΩ, resistor_footprints:R_0402_1005Metric, F.Cu at (144.8, 107.4)
- added R26: 169 kΩ, resistor_footprints:R_0402_1005Metric, F.Cu at (144.8, 105.7)
- added R27: 6.2 kΩ, resistor_footprints:R_0402_1005Metric, F.Cu at (144.8, 108.8)
- moved D5 8.51 mm to (141.3, 110.7), turned to 180 degrees
- moved R8 5.76 mm to (142.4, 109.0), turned to 0 degrees
- moved C5 0.70 mm to (146.8, 102.5)
- moved C18 0.36 mm to (147.8, 110.2)
- moved R17 0.31 mm to (147.2, 108.5)
- moved R16 0.23 mm to (150.0, 109.3)
- moved R15 0.15 mm to (146.7, 106.7)
Connections:
- C2 pad 1: /VIN -> /V_IN
- C3 pad 1: /VIN -> /V_IN
- C4 pad 1: /VIN -> /V_IN
- R8 pad 1: /VIN -> /V_IN
- T1 pad 2: /VIN -> /V_IN
- T1 pad 3: /VIN -> /V_IN
- U1 pad 6: unconnected-(U1-VIN-Pad6) -> /VIN
- U1 pad 7: unconnected-(U1-EN-Pad7) -> /EN
Routing:
- net /VIN: track 0.76 -> 7.00 mm, vias 16 -> 0
- net /EN: track 0.00 -> 3.29 mm
- net Net-(R25-Pad2): track 0.00 -> 3.02 mm
- net /SR1: track 33.6 -> 31.3 mm
- net /V_IN: track 0.00 -> 2.29 mm, vias 0 -> 18
- net Net-(Q5-B): track 1.72 -> 3.00 mm
- net /CS: track 18.9 -> 18.1 mm
- net /VREG1: track 34.5 -> 35.1 mm
- net GND: vias 22 -> 26
- added copper zone on F.Cu, net /V_IN
- added copper zone on In1.Cu, net /V_IN
- removed copper zone on F.Cu, net /VIN
- removed copper zone on In1.Cu, net /VIN

Commit message: backup
Parts:
- moved R2 9.09 mm to (130.6, 90.7), turned to 180 degrees
- moved C13 7.73 mm to (179.7, 101.9), turned to 0 degrees
- moved C15 6.24 mm to (179.7, 93.5), turned to 0 degrees
- moved R5 6.06 mm to (131.8, 92.6), turned to 0 degrees
- moved R4 5.86 mm to (131.1, 94.5), turned to 90 degrees
- moved C16 5.13 mm to (179.7, 99.1), turned to 0 degrees
- moved Q1 4.94 mm to (136.6, 92.1), turned to 0 degrees
- moved C17 4.94 mm to (179.7, 96.3), turned to 0 degrees
- moved R3 4.04 mm to (132.4, 94.5), turned to -90 degrees
- moved C14 2.27 mm to (179.7, 90.7), turned to 0 degrees
- moved C12 1.71 mm to (179.7, 87.9), turned to 0 degrees
- moved C7 0.77 mm to (137.1, 96.3)
- moved C9 0.77 mm to (136.5, 102.0)
- moved D4 0.77 mm to (138.1, 103.4)
- moved Q2 0.77 mm to (138.2, 99.6)
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Routing:
- net /CS: track 18.1 -> 26.4 mm
- net /N_GATE: track 17.6 -> 22.5 mm
- net /VREG1: track 35.1 -> 34.2 mm
- net GNDA: vias 47 -> 50
- net GND: vias 26 -> 34
- net /VOUT: vias 36 -> 31
Other:
- board size 59.7 x 36.8 mm -> 55.9 x 36.8 mm

Commit message: backup
Parts:
- moved D2 3.51 mm to (137.9, 82.8)
- moved C1 1.76 mm to (131.9, 83.1)
- moved D3 1.76 mm to (129.9, 81.6)
- moved L1 1.76 mm to (134.5, 81.9)
- moved R1 1.76 mm to (132.9, 79.9)
- moved C2 1.73 mm to (132.9, 87.8)
- moved C3 1.73 mm to (135.7, 87.8)
- moved C4 1.73 mm to (138.5, 87.8)
- moved R4 1.68 mm to (130.6, 96.1)
- moved R2 1.62 mm to (130.4, 92.3)
- moved R3 1.62 mm to (132.2, 96.1)
- moved C7 1.62 mm to (136.8, 97.9)
- moved C8 1.62 mm to (138.7, 98.7)
- moved C9 1.62 mm to (136.3, 103.6)
- moved D4 1.62 mm to (137.9, 105.0)
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Connections:
- R12 pad 1: /SR2_G -> /SR2
- R12 pad 2: /SR2 -> /SR2_G
Routing:
- net /VREG1: track 34.2 -> 36.6 mm
- net /CS: track 26.4 -> 25.6 mm
- net /P_GATE: track 16.1 -> 16.8 mm
- net /SR1: track 31.3 -> 31.8 mm
- net GNDA: vias 50 -> 113
- net GND: vias 34 -> 96
Other:
- board size 55.9 x 36.8 mm -> 55.9 x 35.6 mm

Commit message: backup
Parts:
- added J1: CLP-104-02-G-D-BE, connector_footprints:CLP-104-02-G-D-BE, F.Cu at (135.3, 117.5)
- added MB2: mouse-bite-50mil-300mil, mouse_bite_footprints:mouse-bite-50mil-300mil, F.Cu at (135.3, 113.7)
- added TP1: TestPoint, test_point_footprints:TestPoint_THTPad_Castelated, F.Cu at (133.4, 113.0)
- added TP2: TestPoint, test_point_footprints:TestPoint_THTPad_Castelated, F.Cu at (134.6, 113.0)
- added TP3: TestPoint, test_point_footprints:TestPoint_THTPad_Castelated, F.Cu at (135.9, 113.0)
- added TP4: TestPoint, test_point_footprints:TestPoint_THTPad_Castelated, F.Cu at (137.2, 113.0)
- added TP5: TestPoint, test_point_footprints:TestPoint_THTPad_Castelated, F.Cu at (176.5, 77.5)
- added TP6: TestPoint, test_point_footprints:TestPoint_THTPad_Castelated, F.Cu at (177.8, 77.5)
- added TP7: TestPoint, test_point_footprints:TestPoint_THTPad_Castelated, F.Cu at (179.1, 77.5)
- added TP8: TestPoint, test_point_footprints:TestPoint_THTPad_Castelated, F.Cu at (180.3, 77.5)
- renumbered C7 to C10, C8 to C11, C16 to C12, C6 to C14, C22 to C15, C23 to C16, C5 to C17, C25 to C18, C24 to C19, C10 to C2, C9 to C20, C20 to C21, C21 to C22, C11 to C23, C19 to C24, C18 to C25, C2 to C3, C3 to C4, C4 to C5, C12 to C6, C14 to C7, C15 to C8, C17 to C9, D5 to D10, D3 to D2, D2 to D3, D6 to D4, D9 to D5, D8 to D6, D4 to D7, D7 to D8, D10 to D9, Q3 to Q1, Q1 to Q2, Q2 to Q3, R10 to R1, R11 to R10, R12 to R11, R6 to R12, R23 to R13, R24 to R14, R26 to R15, R15 to R16, R21 to R17, R22 to R18, R25 to R19, R1 to R2, R14 to R20, R17 to R21, R27 to R22, R8 to R23, R20 to R24, R16 to R25, R19 to R26, R18 to R27, R9 to R3, R13 to R4, R2 to R5, R5 to R6, R4 to R7, R3 to R8, R7 to R9
Routing:
- net GNDA: vias 113 -> 111
- net GND: vias 96 -> 93
Other:
- board size 55.9 x 35.6 mm -> 55.9 x 43.7 mm

Commit message: backup
Parts:
- added J2: CLP-104-02-G-D-BE, connector_footprints:CLP-104-02-G-D-BE, F.Cu at (178.4, 73.0)
- added MB1: mouse-bite-50mil-300mil, mouse_bite_footprints:mouse-bite-50mil-300mil, F.Cu at (178.4, 76.8)
Routing:
- net GNDA: vias 111 -> 120
- net /VOUT: vias 31 -> 41
Other:
- board size 55.9 x 43.7 mm -> 55.9 x 51.8 mm

Commit message: backup
Parts:
- moved R1 2.63 mm to (173.0, 81.4)
- moved R3 2.63 mm to (173.0, 82.7)
- moved R10 2.61 mm to (173.2, 104.6)
- moved R11 2.61 mm to (173.2, 106.0)
- moved MB1 2.54 mm to (178.4, 79.4)
- moved TP5 2.54 mm to (176.5, 80.0)
- moved TP6 2.54 mm to (177.8, 80.0)
- moved TP7 2.54 mm to (179.1, 80.0)
- moved TP8 2.54 mm to (180.3, 80.0)
- moved J2 2.54 mm to (178.4, 75.6)
- moved D4 0.25 mm to (168.0, 84.4)
- moved R4 0.25 mm to (172.1, 84.3)
- moved C2 0.25 mm to (170.4, 84.4)
- moved D5 0.25 mm to (169.6, 87.0)
- moved Q1 0.25 mm to (168.2, 80.7)
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Routing:
- net /SR2_G: track 2.84 -> 5.08 mm, vias 0 -> 2
- net /SR1_G: track 2.85 -> 5.08 mm, vias 0 -> 2
- net /SR1: track 31.8 -> 30.7 mm
- net /SR2: track 21.6 -> 22.7 mm
- net /RT: track 1.80 -> 1.76 mm, vias 1 -> 0
- net GNDA: vias 120 -> 117
Other:
- board size 55.9 x 51.8 mm -> 55.9 x 49.3 mm

Commit message: backup
Parts:
- moved R6 3.66 mm to (129.8, 97.4), turned to 90 degrees
- moved R2 3.06 mm to (130.2, 81.3)
- moved R1 2.93 mm to (170.9, 79.3), turned to -90 degrees
- moved D2 2.88 mm to (131.3, 79.0), turned to 0 degrees
- moved J2 2.54 mm to (178.4, 78.1)
- moved MB1 2.54 mm to (178.4, 81.9)
- moved TP5 2.54 mm to (176.5, 82.5)
- moved TP6 2.54 mm to (177.8, 82.5)
- moved TP7 2.54 mm to (179.1, 82.5)
- moved TP8 2.54 mm to (180.3, 82.5)
- moved R3 2.35 mm to (170.9, 81.5), turned to 90 degrees
- moved C1 2.05 mm to (129.9, 82.8), turned to 0 degrees
- moved R20 1.78 mm to (170.6, 107.6)
- moved C23 1.78 mm to (168.9, 107.6)
- moved D8 1.78 mm to (166.3, 107.6)
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Routing:
- net /CS: track 25.6 -> 21.0 mm
- net /N_GATE: track 22.7 -> 21.7 mm
- net /SR1: track 30.7 -> 29.7 mm
- net /SR1_G: track 5.08 -> 5.67 mm
- net /N_GATE_G: track 3.13 -> 2.59 mm
- net /SR2: track 22.7 -> 22.2 mm
- net GNDA: vias 117 -> 115
- net GND: vias 93 -> 89
Other:
- board size 55.9 x 49.3 mm -> 55.9 x 46.7 mm

Commit message: backup
Parts:
- moved J2 2.54 mm to (178.4, 80.6)
- moved TP5 2.54 mm to (176.5, 85.1)
- moved TP6 2.54 mm to (177.8, 85.1)
- moved TP7 2.54 mm to (179.1, 85.1)
- moved TP8 2.54 mm to (180.3, 85.1)
- moved MB1 2.54 mm to (178.4, 84.5)
- moved C9 2.17 mm to (177.9, 98.5)
- moved C12 2.17 mm to (177.9, 101.3)
- moved C13 2.17 mm to (177.9, 104.1)
- moved C6 2.17 mm to (177.9, 90.1)
- moved C7 2.17 mm to (177.9, 92.9)
- moved C8 2.17 mm to (177.9, 95.7)
- moved C2 0.71 mm to (169.6, 84.4)
- moved R4 0.33 mm to (170.9, 84.3)
Routing:
- net GNDA: vias 115 -> 111
- net GND: vias 89 -> 99
- net /V_IN: vias 18 -> 28
Other:
- board size 55.9 x 46.7 mm -> 55.9 x 44.2 mm
