File: minimal_adp1074/minimal_adp1074.kicad_pcb (KiCad board)
At the start: 4 copper layers, 55.9 x 44.2 mm, 83 parts, among them J1 CLP-104-02-G-D-BE, J2 CLP-104-02-G-D-BE, Q1 40 V, Q2 80 V, Q3 -60 V, Q4 40 V, Q5 150 V, T1 PL160X9-102L-BLD, U1 ADP1074ACCZ-R7

Commit message: backup
Parts:
- T1: value PL160X9-102L-BLD -> PL160X9-102L
