File: minimal_adp1074/minimal_adp1074.kicad_sch (KiCad schematic)
At the start: 0 parts

Commit message: backup
Parts:
- added T1: PL160X9-102L-BLD, transformer_footprints:PL160X9-102L, symbol TRANSFORMERS_PL160X9-102L_DATA_BASE:T_PL160X9-102L-BLD
- added U1: ADP1074ACCZ-R7, analog_devices_footprints:CC-24-6_ADI, symbol UNITED_IC_ADI:U_ADP1074ACCZ-R7
Connections:
- new net: T1.4, T1.5
- new net VIN: T1.2, T1.3

Commit message: backup
Parts:
- added D1, D2: 100 V, diode_footprints:SOD323, symbol DIODES_1N4148WX-TP_DATA_BASE:D_1N4148WX-TP
- added L1: 1000.0 µH, inductor_footprints:CB2518T, symbol INDUCTORS_CB2518T_DATA_BASE:L_CB2518T102K
Connections:
- net GNDA: now reaches U1.21 (AGND2)
- net GNDA: now also U1.22 (PGND2), U1.26 (AGND2)
- net GND: now reaches U1.25 (AGND1)
- net GND: now also U1.3 (PGND1), U1.4 (AGND1)
- net at T1.1: now also D1.2
- net at T1.6: now also D2.2
- new net: D1.1, D2.1, L1.1
Other:
- moved on the sheet: U1

Commit message: backup
Parts:
- added C1: 2.2 µF, capacitor_footprints:C_0805_2012Metric, symbol CAPACITORS_CGA4J1X7R1V_DATA_BASE:C_CGA4J1X7R1V225K125AC
- added C2, C3, C4: 2.2 µF, capacitor_footprints:C_1206_3216Metric, symbol CAPACITORS_KGM31HR71H_DATA_BASE:C_KGM31HR71H225KU
- added D3: 11.0 V, diode_footprints:SOD_123, symbol DIODES_BZT52C_DATA_BASE:D_BZT52C11-7-F
- added Q1: 80 V, transistor_footprints:PowerPAK SO-8 Single, symbol TRANSISTORS_SIR680DP-T1-RE3_DATA_BASE:Q_SIR680DP-T1-RE3
- added R1: 100 Ω, resistor_footprints:R_0402_1005Metric, symbol RESISTORS_ERJ-2RKF_DATA_BASE:R_ERJ-2RKF1000X
Connections:
- net GND: now also D2.2, T1.6, C1.1, C2.2, C3.2, C4.2, D3.2
- net VIN: now also C2.1, C3.1, C4.1
- net N_GATE: now reaches U1.1 (NGATE)
- net N_GATE: now also Q1.4 (G)
- net at T1.4, T1.5: now also Q1.5 (D)
- net V_AUX: now reaches L1.2
- net V_AUX: now also C1.2, R1.1
- new net: D3.1, R1.2
- no-connect marks 0 -> 3

Commit message: backup
Parts:
- added C5, C8, C9: 100 nF, capacitor_footprints:C_0402_1005Metric, symbol CAPACITORS_GCM155R71H_DATA_BASE:C_GCM155R71H104KE02D
- added C6: 2.2 µF, capacitor_footprints:C_0603_1608Metric, symbol CAPACITORS_C1005X5R1V_DATA_BASE:C_C1005X5R1V225M050BC
- added C7: 220 nF, capacitor_footprints:C_0603_1608Metric, symbol CAPACITORS_GCM188R71H_DATA_BASE:C_GCM188R71H224KA64D
- added D4: 100 V, diode_footprints:SOD323, symbol DIODES_1N4148WX-TP_DATA_BASE:D_1N4148WX-TP
- added D5: 11.0 V, diode_footprints:SOD_123, symbol DIODES_BZT52C_DATA_BASE:D_BZT52C11-7-F
- added L2: 2.0 µH, inductor_footprints:IHLP4040DZE_V2, symbol INDUCTORS_IHLP4040DZE__DATA_BASE:L_IHLP4040DZE_2R0M11
- added Q2: -60 V, transistor_footprints:SOT-26, symbol TRANSISTORS_ZXMP6A17E6TA_DATA_BASE:Q_ZXMP6A17E6TA
- added R2: 0.008 Ω, resistor_footprints:R_1206_3216Metric, symbol RESISTORS_PMR18EZPFU_DATA_BASE:R_PMR18EZPFU8L00
- added R3, R6, R8: 10 kΩ, resistor_footprints:R_0402_1005Metric, symbol RESISTORS_ERJ-2RKF_DATA_BASE:R_ERJ-2RKF1002X
- added R4: 0 Ω, resistor_footprints:R_0402_1005Metric, symbol RESISTORS_ERJ-2GE0_DATA_BASE:R_ERJ-2GE0R00X
- added R5: 1.5 kΩ, resistor_footprints:R_0402_1005Metric, symbol RESISTORS_ERJ-2RKF_DATA_BASE:R_ERJ-2RKF1501X
- added R7: 1 kΩ, resistor_footprints:R_0402_1005Metric, symbol RESISTORS_ERJ-2RKF_DATA_BASE:R_ERJ-2RKF1001X
- C1: footprint capacitor_footprints:C_0805_2012Metric -> capacitor_footprints:C_0603_1608Metric; symbol CAPACITORS_CGA4J1X7R1V_DATA_BASE:C_CGA4J1X7R1V225K125AC -> CAPACITORS_C1005X5R1V_DATA_BASE:C_C1005X5R1V225M050BC; Case Code - in 0805 -> 0603; Case Code - mm 2012 -> 1608; Dielectric X7R -> X5R; MPN CGA4J1X7R1V225K125AC -> C1005X5R1V225M050BC; Series CGA4J1X7R1V -> C1005X5R1V; Symbol Name C_CGA4J1X7R1V225K125AC -> C_C1005X5R1V225M050BC; Tolerance 10% -> 20%; Trustedparts Search https://www.trustedparts.com/en/search/CGA4J1X7R1V225K125AC -> https://www.trustedparts.com/en/search/C1005X5R1V225M050BC
Connections:
- net V_AUX is gone; now on net VREG1: C1.2, L1.2, R1.1
- net GND: now also C5.2, D4.1, D5.2, Q2.4 (S), R2.2, R3.2, R6.2
- net GNDA: now also C6.2
- net N_GATE: now also R4.1; no longer Q1.4 (G)
- net VIN: now also R8.1
- net at Q1.1 (S): now also Q1.2 (S), Q1.3 (S), R2.1, R5.2
- net at Q1.5 (D), T1.4, T1.5: now also C7.1, R7.1
- net P_GATE: now reaches U1.2 (PGATE)
- net P_GATE: now also C9.1
- net VERG2: now reaches U1.20 (VREG2)
- net VERG2: now also C6.1
- net VREG1: now reaches U1.5 (VREG1)
- net VREG1: now also C5.1
- net CS: now reaches U1.8 (CS)
- net CS: now also R5.1
- net at T1.7: now also L2.1
- new net: C9.2, D4.2, Q2.3 (G), R6.1
- new net: Q1.4 (G), R3.1, R4.2
- new net: C7.2, C8.2, Q2.1 (D), Q2.2 (D), Q2.5 (D), Q2.6 (D)
- new net: D5.1, R8.2
- new net: C8.1, R7.2
- new net VOUT: L2.2
Other:
- moved on the sheet: C1, C2, C3, C4, D1, D2, D3, L1, Q1, R1, U1

Commit message: backup
Parts:
- added C10, C11: 10 nF, capacitor_footprints:C_0402_1005Metric, symbol CAPACITORS_GCM155R71H_DATA_BASE:C_GCM155R71H103KA55D
- added D6, D7: 100 V, diode_footprints:SOD323, symbol DIODES_1N4148WX-TP_DATA_BASE:D_1N4148WX-TP
- added Q3, Q4: 40 V, transistor_footprints:TDSON-8 FL, symbol TRANSISTORS_BSC014N04LSI_DATA_BASE:Q_BSC014N04LSI
- added R10, R11, R13, R14: 10 kΩ, resistor_footprints:R_0402_1005Metric, symbol RESISTORS_ERJ-2RKF_DATA_BASE:R_ERJ-2RKF1002X
- added R12, R9: 0 Ω, resistor_footprints:R_0402_1005Metric, symbol RESISTORS_ERJ-2GE0_DATA_BASE:R_ERJ-2GE0R00X
- L2: value 2.0 µH -> 2.2 µH; footprint inductor_footprints:IHLP4040DZE_V2 -> inductor_footprints:74439369; symbol INDUCTORS_IHLP4040DZE__DATA_BASE:L_IHLP4040DZE_2R0M11 -> INDUCTORS_74439369_DATA_BASE:L_74439369022; MPN IHLP4040DZE_2R0M11 -> 74439369022; Manufacturer Vishay -> Wurth Elektronik; Maximum DC Current (A) 16.0 -> 32.0; Maximum DC Resistance (Ω) 5.200 -> 2.420; Series IHLP4040DZE_ -> 74439369; Symbol Name L_IHLP4040DZE_2R0M11 -> L_74439369022; Trustedparts Search https://www.trustedparts.com/en/search/IHLP4040DZE_2R0M11 -> https://www.trustedparts.com/en/search/74439369022
Connections:
- net GNDA: now also C10.2, C11.2, Q3.1 (S), Q3.2 (S), Q3.3 (S), Q4.1 (S), Q4.2 (S), Q4.3 (S), R10.2, R11.1
- net VOUT: now also R13.1, R14.1
- net P_GATE_G: now reaches C9.2, D4.2, Q2.3 (G), R6.1
- net N_GATE_G: now reaches Q1.4 (G), R3.1, R4.2
- net SR2: now reaches U1.23 (SR2)
- net SR2: now also R12.2
- net SR1: now reaches U1.24 (SR1)
- net SR1: now also R9.1
- net at L2.1, T1.7: now also D7.2, Q4.5 (D)
- net at T1.11: now also D6.2, Q3.5 (D)
- new net: C11.1, D7.1, R14.2
- new net: C10.1, D6.1, R13.2
- new net SR1_G: Q3.4 (G), R10.1, R9.2
- new net SR2_G: Q4.4 (G), R11.2, R12.1
Other:
- moved on the sheet: L2, R4

Commit message: backup
Parts:
- added C12, C13, C14, C15, C16, C17: 220 µF, capacitor_footprints:C_1206_3216Metric, symbol CAPACITORS_GRM31CR60J_DATA_BASE:C_GRM31CR60J227ME11K
- added C18: 1.5 µF, capacitor_footprints:C_0603_1608Metric, symbol CAPACITORS_C1005X5R1V_DATA_BASE:C_C1005X5R1V155M050BC
- added C19: 100 nF, capacitor_footprints:C_0402_1005Metric, symbol CAPACITORS_GCM155R71H_DATA_BASE:C_GCM155R71H104KE02D
- added C20: 100 pF, capacitor_footprints:C_0402_1005Metric, symbol CAPACITORS_GCM1555C1H_DATA_BASE:C_GCM1555C1H101FA16D
- added C21: 4.7 nF, capacitor_footprints:C_0402_1005Metric, symbol CAPACITORS_GCM155R71H_DATA_BASE:C_GCM155R71H472KA37D
- added R15: 28 kΩ, resistor_footprints:R_0402_1005Metric, symbol RESISTORS_ERJ-2RKF_DATA_BASE:R_ERJ-2RKF2802X
- added R16: 49.9 kΩ, resistor_footprints:R_0402_1005Metric, symbol RESISTORS_ERJ-2RKF_DATA_BASE:R_ERJ-2RKF4992X
- added R17, R19: 0 Ω, resistor_footprints:R_0402_1005Metric, symbol RESISTORS_ERJ-2GE0_DATA_BASE:R_ERJ-2GE0R00X
- added R18: 10 kΩ, resistor_footprints:R_0402_1005Metric, symbol RESISTORS_ERJ-2RKF_DATA_BASE:R_ERJ-2RKF1002X
- added R20: 24.9 kΩ, resistor_footprints:R_0402_1005Metric, symbol RESISTORS_ERJ-2RKF_DATA_BASE:R_ERJ-2RKF2492X
- added R21: 3.16 kΩ, resistor_footprints:R_0402_1005Metric, symbol RESISTORS_ERJ-2RKF_DATA_BASE:R_ERJ-2RKF3161X
- added R22: 976 Ω, resistor_footprints:R_0402_1005Metric, symbol RESISTORS_ERJ-2RKF_DATA_BASE:R_ERJ-2RKF9760X
- added R23: 3.09 kΩ, resistor_footprints:R_0402_1005Metric, symbol RESISTORS_ERJ-2RKF_DATA_BASE:R_ERJ-2RKF3091X
- added R24: 887 Ω, resistor_footprints:R_0402_1005Metric, symbol RESISTORS_ERJ-2RKF_DATA_BASE:R_ERJ-2RKF8870X
Connections:
- net GND: now also C18.2, R16.2, R17.2
- net GNDA: now also C12.2, C13.2, C14.2, C15.2, C16.2, C17.2, C19.2, C20.2, R19.2, R20.2, R22.2, R24.2
- net VOUT: now also C12.1, C13.1, C14.1, C15.1, C16.1, C17.1, R21.2, R23.1
- net SYNC: now reaches U1.10 (SYNC)
- net SYNC: now also R17.1
- net SS1: now reaches U1.11 (SS1)
- net SS1: now also C18.1
- net DMAX: now reaches U1.12 (DMAX)
- net DMAX: now also R15.2, R16.1
- net MODE: now reaches U1.13 (MODE)
- net MODE: now also R19.1
- net ~{PGOOD}: now reaches U1.14 (~{PGOOD})
- net ~{PGOOD}: now also R18.2
- net SS2: now reaches U1.15 (SS2)
- net SS2: now also C19.1
- net COMP: now reaches U1.16 (COMP)
- net COMP: now also C20.1, C21.1
- net FB: now reaches U1.17 (FB)
- net FB: now also R21.1, R22.1
- net OVP: now reaches U1.18 (OVP)
- net OVP: now also R23.2, R24.1
- net RT: now reaches U1.9 (RT)
- net RT: now also R15.1
- net VERG2 renamed VREG2
- net VREG2: now also R18.1
- new net: C21.2, R20.1
Other:
- moved on the sheet: C10, D6, Q1, Q3, R10, R13, R2, R3, R4, R5, R9, U1

Commit message: backup
Parts:
- added C22, C23: 1.5 µF, capacitor_footprints:C_0603_1608Metric, symbol CAPACITORS_C1005X5R1V_DATA_BASE:C_C1005X5R1V155M050BC
- added D10, D9: 40 V, diode_footprints:SMA, symbol DIODES_B240A-13-F_DATA_BASE:D_B240A-13-F
- added D8: 100 V, diode_footprints:SOD323, symbol DIODES_1N4148WX-TP_DATA_BASE:D_1N4148WX-TP
Connections:
- net GNDA: now also C22.2, C23.2, D10.2, D9.2
- net SW: now reaches D7.2, L2.1, Q4.5 (D), T1.7
- net SW: now also D10.1, D8.2
- net VDD2: now reaches U1.19 (VDD2)
- net VDD2: now also C22.1, C23.1, D8.1
- net at D6.2, Q3.5 (D), T1.11: now also D9.1
Other:
- moved on the sheet: C10, C11, C18, C19, C20, C21, C5, C6, D6, D7, Q1, Q3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

Commit message: backup
Other:
- moved on the sheet: C10, C11, C12, C13, C14, C15, C16, C17, D10, D6, D7, D9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
