File: minimal_adp1074/minimal_adp1074.kicad_sch (KiCad schematic)
At the start: 65 parts, among them Q1 80 V, Q2 -60 V, Q3 40 V, Q4 40 V, T1 PL160X9-102L-BLD, U1 ADP1074ACCZ-R7

Commit message: backup
Parts:
- added C24, C25: 2.2 µF, capacitor_footprints:C_0603_1608Metric, symbol CAPACITORS_C1005X5R1V_DATA_BASE:C_C1005X5R1V225M050BC
- added Q5: 150 V, transistor_footprints:SOT23-3, symbol TRANSISTORS_FMMT625TA_DATA_BASE:Q_FMMT625TA
- added R25: 24.3 kΩ, resistor_footprints:R_0402_1005Metric, symbol RESISTORS_ERJ-2RKF_DATA_BASE:R_ERJ-2RKF2432X
- added R26: 169 kΩ, resistor_footprints:R_0402_1005Metric, symbol RESISTORS_ERJ-2RKF_DATA_BASE:R_ERJ-2RKF1693X
- added R27: 6.2 kΩ, resistor_footprints:R_0402_1005Metric, symbol RESISTORS_ERJ-2RKF_DATA_BASE:R_ERJ-2RKF6201X
Connections:
- net GND: now also C24.2, C25.2, R27.2
- net VIN: now also U1.6 (VIN), C24.1, C25.1, Q5.2 (E); no longer C2.1, C3.1, C4.1, R8.1, T1.2, T1.3
- net EN: now reaches U1.7 (EN)
- net EN: now also R26.2
- net at D5.1, R8.2: now also Q5.1 (B)
- new net: R25.2, R26.1, R27.1
- new net V_IN: C2.1, C3.1, C4.1, Q5.3 (C), R25.1, R8.1, T1.2, T1.3
Other:
- moved on the sheet: C18, C19, C20, C21, D5, Q1, R15, R16, R17, R18, R19, R2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

Commit message: backup
Other:
- moved on the sheet: C7, C8, C9, D4, Q1, Q2, R2, R3, R4, R5, R6, R7

Commit message: backup
Connections:
- net SR2: now also R12.1; no longer R12.2
- net SR2_G: now also R12.2; no longer R12.1
Other:
- moved on the sheet: C10, C11, C12, C13, C14, C15, C16, C17, C18, C19, C20, C21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

Commit message: backup
Parts:
- added J1: CLP-104-02-G-D-BE, connector_footprints:CLP-104-02-G-D-BE, symbol UNITED_CONNECTORS_DATA_BASE:J_CLP-104-02-G-D-BE
- added MB2: mouse-bite-50mil-300mil, mouse_bite_footprints:mouse-bite-50mil-300mil, symbol UNITED_MOUSE_BITES_DATA_BASE:mouse-bite-50mil-300mil
- added TP1, TP2, TP3, TP4, TP5, TP6, TP7, TP8: TestPoint, test_point_footprints:TestPoint_THTPad_Castelated, symbol UNITED_TEST_POINTS:TestPoint_Castelated_v2
- renumbered C7 to C10, C8 to C11, C16 to C12, C6 to C14, C22 to C15, C23 to C16, C5 to C17, C25 to C18, C24 to C19, C10 to C2, C9 to C20, C20 to C21, C21 to C22, C11 to C23, C19 to C24, C18 to C25, C2 to C3, C3 to C4, C4 to C5, C12 to C6, C14 to C7, C15 to C8, C17 to C9, D5 to D10, D3 to D2, D2 to D3, D6 to D4, D9 to D5, D8 to D6, D4 to D7, D7 to D8, D10 to D9, Q3 to Q1, Q1 to Q2, Q2 to Q3, R10 to R1, R11 to R10, R12 to R11, R6 to R12, R23 to R13, R24 to R14, R26 to R15, R15 to R16, R21 to R17, R22 to R18, R25 to R19, R1 to R2, R14 to R20, R17 to R21, R27 to R22, R8 to R23, R20 to R24, R16 to R25, R19 to R26, R18 to R27, R9 to R3, R13 to R4, R2 to R5, R5 to R6, R4 to R7, R3 to R8, R7 to R9
Connections:
- net GND: now also J1.5, J1.6, J1.7, J1.8, TP3.1, TP4.1
- net GNDA: now also TP7.1, TP8.1
- net VOUT: now also TP5.1, TP6.1
- net V_IN: now also J1.1, J1.2, J1.3, J1.4, TP1.1, TP2.1

Commit message: backup
Parts:
- added J2: CLP-104-02-G-D-BE, connector_footprints:CLP-104-02-G-D-BE, symbol UNITED_CONNECTORS_DATA_BASE:J_CLP-104-02-G-D-BE
- added MB1: mouse-bite-50mil-300mil, mouse_bite_footprints:mouse-bite-50mil-300mil, symbol UNITED_MOUSE_BITES_DATA_BASE:mouse-bite-50mil-300mil
Connections:
- net GNDA: now also J2.5, J2.6, J2.7, J2.8
- net VOUT: now also J2.1, J2.2, J2.3, J2.4
Other:
- moved on the sheet: C1, C10, C11, C12, C13, C14, C15, C16, C17, C18, C19, C2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

Commit message: backup
Parts:
- T1: value PL160X9-102L-BLD -> PL160X9-102L; symbol TRANSFORMERS_PL160X9-102L_DATA_BASE:T_PL160X9-102L-BLD -> TRANSFORMERS_PL160X9-102L_DATA_BASE:T_PL160X9-102L; MPN PL160X9-102L-BLD -> PL160X9-102L; Symbol Name T_PL160X9-102L-BLD -> T_PL160X9-102L; Trustedparts Search https://www.trustedparts.com/en/search/PL160X9-102L-BLD -> https://www.trustedparts.com/en/search/PL160X9-102L
Changed lines of the file:
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@@
 	)
 	(symbol
-		(lib_id "TRANSFORMERS_PL160X9-102L_DATA_BASE:T_PL160X9-102L-BLD")
+		(lib_id "TRANSFORMERS_PL160X9-102L_DATA_BASE:T_PL160X9-102L")
 		(at 157.48 101.6 0)
 		(unit 1)
@@
 			)
 		)
-		(property "Value" "PL160X9-102L-BLD"
+		(property "Value" "PL160X9-102L"
 			(at 157.48 78.74 0)
 			(effects
@@
 			)
 		)
-		(property "MPN" "PL160X9-102L-BLD"
+		(property "MPN" "PL160X9-102L"
 			(at 157.48 134.62 0)
 			(show_name yes)
@@
 			)
 		)
-		(property "Symbol Name" "T_PL160X9-102L-BLD"
+		(property "Symbol Name" "T_PL160X9-102L"
 			(at 157.48 147.32 0)
 			(show_name yes)
@@
 			)
 		)
-		(property "Trustedparts Search" "https://www.trustedparts.com/en/search/PL160X9-102L-BLD"
+		(property "Trustedparts Search" "https://www.trustedparts.com/en/search/PL160X9-102L"
 			(at 157.48 152.4 0)
 			(show_name yes)
